File: PCBWay/PCBWay.kicad_pcb (KiCad board)
At the start: 2 copper layers, 0 parts

Commit message: Give PCBWay a copy of the JLCPCB test board
The PCBWay board was empty, so its rules had never run against anything. This is the JLCPCB board and schematic copied over, with PCBWay's own project file kept; the object types match the rule set. Tuning the pass/fail objects to PCBWay's values is still open. CI no longer needs to borrow the JLCPCB board for PCBWay.

Refs #14
Parts:
- added ?: , , F.Cu at (143.9, 126.6)
- added ?: , , F.Cu at (143.0, 126.6)
- added ?: , , F.Cu at (121.0, 187.0)
- added ?: , , F.Cu at (145.1, 187.0)
- added ?: , , F.Cu at (119.0, 126.5)
- added ?: , , F.Cu at (120.0, 126.5)
- added R1: 1k, Resistor_THT:R_Axial_DIN0204_L3.6mm_D1.6mm_P2.54mm_Vertical, F.Cu at (129.0, 17.0)
- added REF**: R_0805_2012Metric, Resistor_SMD:R_0805_2012Metric, F.Cu at (143.0, 79.0)
- added REF**: MountingHole_2.1mm, MountingHole:MountingHole_2.1mm, F.Cu at (119.0, 110.0)
- added REF**: R_0805_2012Metric, Resistor_SMD:R_0805_2012Metric, F.Cu at (121.0, 79.0)
- added REF**: Pin_D0.7mm_L6.5mm_W1.8mm_FlatFork, Connector_Pin:Pin_D0.7mm_L6.5mm_W1.8mm_FlatFork, F.Cu at (143.0, 159.9)
- added REF**: MountingHole_2.2mm_M2_DIN965_Pad_TopBottom, MountingHole:MountingHole_2.2mm_M2_DIN965_Pad_TopBottom, F.Cu at (143.0, 149.0)
- added REF**: MountingHole_2.2mm_M2_DIN965_Pad_TopBottom, MountingHole:MountingHole_2.2mm_M2_DIN965_Pad_TopBottom, F.Cu at (143.0, 189.0)
- added REF**: MountingHole_2.2mm_M2_DIN965_Pad_TopBottom, MountingHole:MountingHole_2.2mm_M2_DIN965_Pad_TopBottom, F.Cu at (145.2, 189.0)
- added REF**: MountingHole_2.2mm_M2_DIN965_Pad_TopBottom, MountingHole:MountingHole_2.2mm_M2_DIN965_Pad_TopBottom, F.Cu at (123.0, 189.0)
- added REF**: MountingHole_2.2mm_M2_DIN965_Pad_TopBottom, MountingHole:MountingHole_2.2mm_M2_DIN965_Pad_TopBottom, F.Cu at (123.0, 139.0)
- added REF**: MountingHole_2.2mm_M2_DIN965_Pad_TopBottom, MountingHole:MountingHole_2.2mm_M2_DIN965_Pad_TopBottom, F.Cu at (123.0, 169.8)
- added REF**: MountingHole_2.2mm_M2_DIN965_Pad_TopBottom, MountingHole:MountingHole_2.2mm_M2_DIN965_Pad_TopBottom, F.Cu at (120.9, 189.0)
- added REF**: MountingHole_2.2mm_M2_DIN965_Pad_TopBottom, MountingHole:MountingHole_2.2mm_M2_DIN965_Pad_TopBottom, F.Cu at (141.0, 99.0)
- added REF**: MountingHole_2.2mm_M2_DIN965_Pad_TopBottom, MountingHole:MountingHole_2.2mm_M2_DIN965_Pad_TopBottom, F.Cu at (117.0, 129.0)
- added REF**: MountingHole_2.2mm_M2_DIN965_Pad_TopBottom, MountingHole:MountingHole_2.2mm_M2_DIN965_Pad_TopBottom, F.Cu at (124.0, 99.0)
- added REF**: MountingHole_3.5mm_Pad_TopBottom, MountingHole:MountingHole_3.5mm_Pad_TopBottom, F.Cu at (146.0, 99.0)
- added REF**: MountingHole_2.1mm, MountingHole:MountingHole_2.1mm, F.Cu at (146.0, 110.0)
- added REF**: MountingHole_2.2mm_M2_DIN965_Pad_TopBottom, MountingHole:MountingHole_2.2mm_M2_DIN965_Pad_TopBottom, F.Cu at (123.0, 179.2)
- added REF**: MountingHole_2.2mm_M2_DIN965_Pad_TopBottom, MountingHole:MountingHole_2.2mm_M2_DIN965_Pad_TopBottom, F.Cu at (123.0, 149.0)
- added REF**: MountingHole_2.2mm_M2_DIN965_Pad_TopBottom, MountingHole:MountingHole_2.2mm_M2_DIN965_Pad_TopBottom, F.Cu at (145.0, 129.0)
- added REF**: MountingHole_3.7mm_Pad_TopBottom, MountingHole:MountingHole_3.7mm_Pad_TopBottom, F.Cu at (119.0, 99.0)
- added REF**: MountingHole_2.2mm_M2_DIN965_Pad_TopBottom, MountingHole:MountingHole_2.2mm_M2_DIN965_Pad_TopBottom, F.Cu at (143.0, 139.0)
- added REF**: MountingHole_2.2mm_M2_DIN965_Pad_TopBottom, MountingHole:MountingHole_2.2mm_M2_DIN965_Pad_TopBottom, F.Cu at (143.0, 179.3)
- added REF**: MountingHole_2.2mm_M2_DIN965_Pad_TopBottom, MountingHole:MountingHole_2.2mm_M2_DIN965_Pad_TopBottom, F.Cu at (128.0, 119.0)
- added REF**: MountingHole_2.2mm_M2_DIN965_Pad_TopBottom, MountingHole:MountingHole_2.2mm_M2_DIN965_Pad_TopBottom, F.Cu at (143.0, 169.9)
- added REF**: Pin_D0.7mm_L6.5mm_W1.8mm_FlatFork, Connector_Pin:Pin_D0.7mm_L6.5mm_W1.8mm_FlatFork, F.Cu at (123.0, 159.8)
- added REF**: MountingHole_2.2mm_M2_DIN965_Pad_TopBottom, MountingHole:MountingHole_2.2mm_M2_DIN965_Pad_TopBottom, F.Cu at (135.0, 119.0)
Routing:
- net GND: track 0.00 -> 696.4 mm, vias 0 -> 8
- net +5V: track 0.00 -> 469.0 mm, vias 0 -> 11
- net (no net): vias 0 -> 4
Other:
- board outline added: 180 x 235 mm
- copper layers 2 -> 4
- board text added: "FAIL"
- board text added: "Just big and thick enough"
- board text added: "PASS"
- board text added: "Too small"
- board text added: "Too thin"
